File: hardware/KiCad/chain_counter.kicad_sch (KiCad schematic)
At the start: 39 parts

Commit message: doco and hardware design fix
Parts:
- added J1: 6P4C, symbol Connector:6P4C
Connections:
- net SW_Down: now also U?.37 (IO23); no longer U?.8 (IO32)
- net SW_Up: now also U?.8 (IO32); no longer U?.37 (IO23)
